Commit message: Added fake freedrive script, and added my end effector to robot cell

File: cell/my_robot_cell_description/urdf/my_robot_cell_macro.xacro (robot description, xacro)
@@ -34,5 +34,5 @@
         </geometry>
         <!-- TODO, measure how thick and how far in on the real table the mounting plate is-->
-        <origin xyz="-0.5 0 -0.020" rpy="0 0 0"/>
+        <origin xyz="-0.5 0 -0.020" rpy="0 0 ${pi/2}"/>
       </collision>
     </link>
@@ -70,15 +70,21 @@
             </material>
             <geometry>
-                <cylinder length="0.125" radius="0.0125"/>
+                <mesh filename="package://my_robot_cell_description/meshes/CustomEndEffector.stl"/>
             </geometry>
-            <origin xyz="0 0 0.0625"/>
+            <origin rpy="${pi} 0 0" xyz="0 0 0"/>
         </visual>
         <collision>
             <geometry>
-                <cylinder length="0.125" radius="0.0125"/>
+                <mesh filename="package://my_robot_cell_description/meshes/CustomEndEffector.stl"/>
             </geometry>
-            <origin xyz="0 0 0.0625"/>
+            <origin rpy="${pi} 0 0" xyz="0 0 0"/>
         </collision>
     </link>
+    <joint name="end_effector_to_tip" type="fixed">
+        <parent link="end_effector"/>
+        <child link="tip"/>
+        <origin xyz="0 0 0.044"/>
+    </joint>
+    <link name="tip"/>
   </xacro:macro>
 </robot>

Commit message: almost there, just need to make it move WRT the tip, rather than the 'end effector'

File: cell/my_robot_cell_description/urdf/my_robot_cell_macro.xacro (robot description, xacro)
@@ -34,5 +34,5 @@
         </geometry>
         <!-- TODO, measure how thick and how far in on the real table the mounting plate is-->
-        <origin xyz="-0.5 0 -0.020" rpy="0 0 ${pi/2}"/>
+        <origin xyz="-0.5 0 -0.020" rpy="0 0 0"/>
       </collision>
     </link>
@@ -40,5 +40,5 @@
       <parent link="table"/>
       <child link="robot_mount"/>
-      <origin xyz="-0.15 0 0.025" rpy="0 0 ${pi}" />
+      <origin xyz="-0.15 0 0.025" rpy="0 0 ${pi/2}" />
     </joint>
     <!-- Link that joins OUR stuff, to the robot -->
